Commit message: testing with coupled sensors

File: urdf/my_robot.urdf (robot description, URDF)
Before this commit: robot test_robot, 4 links, 3 joints
Links:
- removed link link1
- removed link link2
- removed link link3
- removed link link4
Joints:
- removed joint joint1
- removed joint joint2
- removed joint joint3
